Commit message: Changed robot model to a F1 car!

File: urdf/udacity_bot.xacro (robot description, xacro)
@@ -22,11 +22,35 @@
       <origin xyz="0 0 0" rpy=" 0 0 0"/>
       <geometry>
-        <box size=".4 .2 .1"/>
-      </geometry>
-    </collision>
-    <visual name='chassis_visual'>
-      <origin xyz="0 0 0" rpy=" 0 0 0"/>
-      <geometry>
-        <box size=".4 .2 .1"/>
+        <box size=".5 .2 .1"/>
+      </geometry>
+    </collision>
+    <visual name='base_chassis_visual'>
+      <origin xyz="-0.1 0 -0.025" rpy=" 0 0 0"/>
+      <geometry>
+        <box size=".2 .2 .05"/>
+      </geometry>
+    </visual>
+    <visual name='top_chassis_visual'>
+      <origin xyz="-0.1 0 0.03" rpy=" 0 0 0"/>
+      <geometry>
+        <box size=".2 .1 .06"/>
+      </geometry>
+    </visual>
+    <visual name='front_chassis_visual'>
+      <origin xyz="0.1 0 -0.025" rpy=" 0 0 0"/>
+      <geometry>
+        <box size=".2 .1 .05"/>
+      </geometry>
+    </visual>
+    <visual name='front_wing_visual'>
+      <origin xyz="0.2 0 -0.04" rpy=" 0 0 0"/>
+      <geometry>
+        <box size=".1 .3 0.02"/>
+      </geometry>
+    </visual>
+     <visual name='rear_wing_visual'>
+      <origin xyz="-0.2 0 0.1" rpy=" 0 0 0"/>
+      <geometry>
+        <box size=".1 .3 0.02"/>
       </geometry>
     </visual>
@@ -162,5 +186,5 @@
   </link>
   <joint type="fixed" name="camera_joint">
-    <origin xyz="0.2 0 0" rpy="0 0 0"/>
+    <origin xyz="0.025 0 0.025" rpy="0 0 0"/>
     <child link="camera"/>
     <parent link="chassis"/>
@@ -190,5 +214,5 @@
   </link>
   <joint type="fixed" name="hokuyo_joint">
-    <origin xyz=".15 0 .1" rpy="0 0 0"/>
+    <origin xyz="-.05 0 .1" rpy="0 0 0"/>
     <child link="hokuyo"/>
     <parent link="chassis"/>

Commit message: Final changes before first submission

File: urdf/udacity_bot.xacro (robot description, xacro)
@@ -41,16 +41,4 @@
       <geometry>
         <box size=".2 .1 .05"/>
-      </geometry>
-    </visual>
-    <visual name='front_wing_visual'>
-      <origin xyz="0.2 0 -0.04" rpy=" 0 0 0"/>
-      <geometry>
-        <box size=".1 .3 0.02"/>
-      </geometry>
-    </visual>
-     <visual name='rear_wing_visual'>
-      <origin xyz="-0.2 0 0.1" rpy=" 0 0 0"/>
-      <geometry>
-        <box size=".1 .3 0.02"/>
       </geometry>
     </visual>
@@ -100,4 +88,30 @@
     </visual>
   </link>
+  <link name="front_wing">
+      <visual name='front_wing_visual'>
+      <origin xyz="0 0 0" rpy=" 0 0 0"/>
+      <geometry>
+        <box size=".1 .3 0.02"/>
+      </geometry>
+    </visual>
+  </link>
+  <joint type="fixed" name="front_wing_joint">
+    <origin xyz="0.2 0 -0.04" rpy=" 0 0 0"/>
+    <child link="front_wing"/>
+    <parent link="chassis"/>
+  </joint>
+  <link name="rear_wing">
+     <visual name='rear_wing_visual'>
+      <origin xyz="0 0 0" rpy=" 0 0 0"/>
+      <geometry>
+        <box size=".1 .3 0.02"/>
+      </geometry>
+    </visual>
+  </link>
+  <joint type="fixed" name="rear_wing_joint">
+    <origin xyz="-0.2 0 0.1" rpy=" 0 0 0"/>
+    <child link="rear_wing"/>
+    <parent link="chassis"/>
+  </joint>
   <link name="left_wheel">
     <inertial>

Commit message: Created separate xacro file for F1 Model

File: urdf/udacity_bot.xacro (robot description, xacro)
@@ -22,23 +22,11 @@
       <origin xyz="0 0 0" rpy=" 0 0 0"/>
       <geometry>
-        <box size=".5 .2 .1"/>
+        <box size=".4 .2 .1"/>
       </geometry>
     </collision>
-    <visual name='base_chassis_visual'>
-      <origin xyz="-0.1 0 -0.025" rpy=" 0 0 0"/>
+    <visual name='chassis_visual'>
+      <origin xyz="0 0 0" rpy=" 0 0 0"/>
       <geometry>
-        <box size=".2 .2 .05"/>
-      </geometry>
-    </visual>
-    <visual name='top_chassis_visual'>
-      <origin xyz="-0.1 0 0.03" rpy=" 0 0 0"/>
-      <geometry>
-        <box size=".2 .1 .06"/>
-      </geometry>
-    </visual>
-    <visual name='front_chassis_visual'>
-      <origin xyz="0.1 0 -0.025" rpy=" 0 0 0"/>
-      <geometry>
-        <box size=".2 .1 .05"/>
+        <box size=".4 .2 .1"/>
       </geometry>
     </visual>
@@ -88,30 +76,4 @@
     </visual>
   </link>
-  <link name="front_wing">
-      <visual name='front_wing_visual'>
-      <origin xyz="0 0 0" rpy=" 0 0 0"/>
-      <geometry>
-        <box size=".1 .3 0.02"/>
-      </geometry>
-    </visual>
-  </link>
-  <joint type="fixed" name="front_wing_joint">
-    <origin xyz="0.2 0 -0.04" rpy=" 0 0 0"/>
-    <child link="front_wing"/>
-    <parent link="chassis"/>
-  </joint>
-  <link name="rear_wing">
-     <visual name='rear_wing_visual'>
-      <origin xyz="0 0 0" rpy=" 0 0 0"/>
-      <geometry>
-        <box size=".1 .3 0.02"/>
-      </geometry>
-    </visual>
-  </link>
-  <joint type="fixed" name="rear_wing_joint">
-    <origin xyz="-0.2 0 0.1" rpy=" 0 0 0"/>
-    <child link="rear_wing"/>
-    <parent link="chassis"/>
-  </joint>
   <link name="left_wheel">
     <inertial>
@@ -200,5 +162,5 @@
   </link>
   <joint type="fixed" name="camera_joint">
-    <origin xyz="0.025 0 0.025" rpy="0 0 0"/>
+    <origin xyz="0.2 0 0" rpy="0 0 0"/>
     <child link="camera"/>
     <parent link="chassis"/>
@@ -228,5 +190,5 @@
   </link>
   <joint type="fixed" name="hokuyo_joint">
-    <origin xyz="-.05 0 .1" rpy="0 0 0"/>
+    <origin xyz=".15 0 .1" rpy="0 0 0"/>
     <child link="hokuyo"/>
     <parent link="chassis"/>
